File: KiCad_Project/FlightPad/_autosave-FlightPad.kicad_pcb (KiCad board)
At the start: 2 copper layers, 70.5 x 94 mm, 20 parts, among them J1 Conn_01x04_Pin, SW10 SW_Push, SW2 SW_Push, SW3 SW_Push, SW4 SW_Push, SW5 SW_Push, SW6 SW_Push, SW7 SW_Push, SW8 SW_Push, SW9 SW_Push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

Commit message: Did the case
Routing:
- net (no net): vias 2 -> 0
Other:
- outline, holes or cut-outs redrawn
Changed lines of the file:
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@@
 		)
 		(property "Value" "Conn_01x04_Pin"
-			(at 18.5 14 360)
+			(at 18.5 14 0)
 			(layer "F.Fab")
 			(effects
@@
 		)
 		(property "Footprint" "KiCad-SSD1306-0.91-OLED-4pin-128x32:SSD1306-0.91-OLED-4pin-128x32"
-			(at 0 0 360)
+			(at 0 0 0)
 			(layer "F.Fab")
 			(hide yes)
@@
 		)
 		(property "Datasheet" ""
-			(at 0 0 360)
+			(at 0 0 0)
 			(layer "F.Fab")
 			(hide yes)
@@
 		)
 		(property "Description" "Generic connector, single row, 01x04, script generated"
-			(at 0 0 360)
+			(at 0 0 0)
 			(layer "F.Fab")
 			(hide yes)
@@
 		)
 		(fp_text user "OLED Panel"
-			(at 18.885 5.885 360)
+			(at 18.885 5.885 0)
 			(layer "F.SilkS")
 			(effects
@@
 		(layer "Edge.Cuts")
 	)
+	(gr_circle
+		(center 118 122)
+		(end 119.5 121)
+		(stroke
+			(width 0.05)
+			(type default)
+		)
+		(fill none)
+		(layer "Edge.Cuts")
+	)
 	(gr_line
 		(start 117 32)
@@
 		(layer "Edge.Cuts")
 	)
+	(gr_circle
+		(center 64.5 38.5)
+		(end 66.5 38)
+		(stroke
+			(width 0.05)
+			(type default)
+		)
+		(fill none)
+		(layer "Edge.Cuts")
+	)
 	(gr_line
 		(start 103.5 35.5)
@@
 		(layer "Edge.Cuts")
 	)
+	(gr_circle
+		(center 56.5 121.5)
+		(end 58 120.5)
+		(stroke
+			(width 0.05)
+			(type default)
+		)
+		(fill none)
+		(layer "Edge.Cuts")
+	)
 	(gr_arc
 		(start 117 32)
@@
 		(layer "Edge.Cuts")
 	)
-	(via
-		(at 118 121)
-		(size 4)
-		(drill 3.4)
-		(layers "F.Cu" "B.Cu")
-		(net 0)
-	)
-	(via
-		(at 55.5 121.5)
-		(size 4)
-		(drill 3.4)
-		(layers "F.Cu" "B.Cu")
-		(net 0)
-	)
 	(segment
