File: KiCad_Project/FlightPad/FlightPad.kicad_pcb (KiCad board)
At the start: 2 copper layers, 70.5 x 94 mm, 20 parts, among them J1 Conn_01x04_Pin, SW10 SW_Push, SW2 SW_Push, SW3 SW_Push, SW4 SW_Push, SW5 SW_Push, SW6 SW_Push, SW7 SW_Push, SW8 SW_Push, SW9 SW_Push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

Commit message: Added More Pics
Routing:
- net (no net): vias 2 -> 0
Other:
- outline, holes or cut-outs redrawn
- board text added: "Designed By Lawri Darbyshire in the UK"
- board text added: "Key Matrix"
- board text added: "Third Screw Hole for Open Top Design"
Changed lines of the file:
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@@
 		)
 		(property "Value" "Conn_01x04_Pin"
-			(at 18.5 14 360)
+			(at 19.385 8.885 0)
 			(layer "F.Fab")
 			(effects
@@
 		)
 		(property "Footprint" "KiCad-SSD1306-0.91-OLED-4pin-128x32:SSD1306-0.91-OLED-4pin-128x32"
-			(at 0 0 360)
+			(at 0 0 0)
 			(layer "F.Fab")
 			(hide yes)
@@
 		)
 		(property "Datasheet" ""
-			(at 0 0 360)
+			(at 0 0 0)
 			(layer "F.Fab")
 			(hide yes)
@@
 		)
 		(property "Description" "Generic connector, single row, 01x04, script generated"
-			(at 0 0 360)
+			(at 0 0 0)
 			(layer "F.Fab")
 			(hide yes)
@@
 		)
 		(fp_text user "OLED Panel"
-			(at 18.885 5.885 360)
+			(at 18.885 5.885 0)
 			(layer "F.SilkS")
 			(effects
@@
 	)
 	(gr_line
-		(start 100.5 55.5)
-		(end 115.5 55.5)
+		(start 97 55.5)
+		(end 112 55.5)
 		(stroke
 			(width 0.2)
@@
 		(net 3)
 	)
+	(gr_rect
+		(start 56.5 59)
+		(end 116 119)
+		(stroke
+			(width 0.1)
+			(type default)
+		)
+		(fill none)
+		(layer "F.SilkS")
+	)
+	(gr_rect
+		(start 70.5 120)
+		(end 105 124)
+		(stroke
+			(width 0.1)
+			(type default)
+		)
+		(fill none)
+		(layer "F.SilkS")
+	)
 	(gr_line
 		(start 112.5 32)
@@
 		(layer "Edge.Cuts")
 	)
+	(gr_circle
+		(center 118 122)
+		(end 119.5 121)
+		(stroke
+			(width 0.05)
+			(type default)
+		)
+		(fill none)
+		(layer "Edge.Cuts")
+	)
 	(gr_line
 		(start 117 32)
@@
 		(layer "Edge.Cuts")
 	)
+	(gr_circle
+		(center 64.5 38.5)
+		(end 66.5 38)
+		(stroke
+			(width 0.05)
+			(type default)
+		)
+		(fill none)
+		(layer "Edge.Cuts")
+	)
 	(gr_line
 		(start 103.5 35.5)
@@
 		(layer "Edge.Cuts")
 	)
+	(gr_circle
+		(center 56.5 121.5)
+		(end 58 120.5)
+		(stroke
+			(width 0.05)
+			(type default)
+		)
+		(fill none)
+		(layer "Edge.Cuts")
+	)
 	(gr_arc
 		(start 117 32)
@@
 		(layer "Edge.Cuts")
 	)
-	(via
-		(at 118 121)
-		(size 4)
-		(drill 3.4)
-		(layers "F.Cu" "B.Cu")
-		(net 0)
-	)
-	(via
-		(at 55.5 121.5)
-		(size 4)
-		(drill 3.4)
-		(layers "F.Cu" "B.Cu")
-		(net 0)
+	(gr_text "Key Matrix"
+		(at 81 58.5 0)
+		(layer "F.SilkS")
+		(effects
+			(font
+				(size 1 1)
+				(thickness 0.1)
+			)
+			(justify left bottom)
+		)
+	)
+	(gr_text "Third Screw Hole for Open Top Design"
+		(at 68 38.5 0)
+		(layer "F.SilkS")
+		(effects
+			(font
+				(size 1 1)
+				(thickness 0.1)
+			)
+			(justify left bottom)
+		)
+	)
+	(gr_text "Designed By Lawri Darbyshire in the UK"
+		(at 72 122.5 0)
+		(layer "F.SilkS")
+		(effects
+			(font
+				(size 1 1)
+				(thickness 0.1)
+			)
+			(justify left bottom)
+		)
 	)
 	(segment
